File: ExternalEnclosure.kicad_sch (KiCad schematic)
At the start: 81 parts, among them J1 Molex 0472861001, J2 Molex 0472861001, J3 Molex 0472861001, J4 Molex 0472861001, U1 XC6206P332MR-G, U2 SY6280AAC, U3 GL852G-OHY60_C7501404, U4 CH32V003F4U6, U5 SY6280AAC, X1 12MHz

Commit message: Add back side SMT header for power profiling
Parts:
- added J5: Power Profiling, Connector_PinHeader_2.54mm:PinHeader_2x03_P2.54mm_Vertical_SMD, symbol Connector_Generic:Conn_02x03_Odd_Even
- added NT1, NT2: NetTie_2, NetTie:NetTie-2_SMD_Pad0.5mm, symbol Device:NetTie_2
Connections:
- net +3.3VP: now also J5.2 (Pin_2), NT2.2; no longer C18.1, C20.1, D6.5 (VBUS), J4.1 (Pin_1)
- net +5VP: now also J5.4 (Pin_4), NT1.2; no longer C17.1, C19.1, D5.5 (VBUS), J4.4 (Pin_4)
- net GND: now also J5.5 (Pin_5), J5.6 (Pin_6)
- new net: C17.1, C19.1, D5.5 (VBUS), J4.4 (Pin_4), J5.3 (Pin_3), NT1.1
- new net: C18.1, C20.1, D6.5 (VBUS), J4.1 (Pin_1), J5.1 (Pin_1), NT2.1

Commit message: Tweak bottom clearances, change to slot for magnets on PCB
The bottom clearances weren't quite right around the pogo pin area, and
although my own PCBs made appropriate contact with the pogo pins, the
official Framework LED Matrix input module was about 1mm (!) short of
proper contact with the pins/magnet.  A couple of things:
* My "5mm diameter x 2mm thick" magnets were actually only 1.6mm thick
* It appears that we need an extra 0.5mm clearance between the "thick
  component" area and the pogo pin area.  The nominal clearance here is
  0.4mm but the Framework-supplied module was contacting here.
* The pogo pin plane should have been measured from the PCB bottom,
  which is 0.5mm above the "spacer bottom" level.

That last adjustment also moved the USB connector up by proxy, so we
needed to add a little bit of a bump over it to ensure a reasonable
minimum width for the shell here.  It's possible we'll remove the top
entirely here and fold this into the lid, but that complicates printing
the lid on a FDM 3d printer because the lid top is no longer planer. So
leave it as-is with a bit of a bump for now.

I also adjusted the cutout in the case so that it would accomodate the
original PCB design as well as the new one, since I have 5 perfectly
functional v1 boards.

The magnets also weren't very grabby.  This is party because they were
too far away from the steel (see above) but I decided to beef this up as
well.  Looking at the FW16 midplate it appears that a pair of opposite
polarity magnets is used.  Switch to an oval slot on the PCB so that we
can use a pair of magnets in our version as well.
Parts:
- H1, H10, H2, H9: footprint ExternalMount:MountingHole_5mm_no_keepout -> ExternalMount:MountingHole_5mm_slot_no_keepout
Changed lines of the file:
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@@
 			)
 		)
-		(property "Footprint" "ExternalMount:MountingHole_5mm_no_keepout"
+		(property "Footprint" "ExternalMount:MountingHole_5mm_slot_no_keepout"
 			(at 330.2 44.45 0)
 			(effects
@@
 			)
 		)
-		(property "Footprint" "ExternalMount:MountingHole_5mm_no_keepout"
+		(property "Footprint" "ExternalMount:MountingHole_5mm_slot_no_keepout"
 			(at 330.2 134.62 0)
 			(effects
@@
 			)
 		)
-		(property "Footprint" "ExternalMount:MountingHole_5mm_no_keepout"
+		(property "Footprint" "ExternalMount:MountingHole_5mm_slot_no_keepout"
 			(at 330.2 39.37 0)
 			(effects
@@
 			)
 		)
-		(property "Footprint" "ExternalMount:MountingHole_5mm_no_keepout"
+		(property "Footprint" "ExternalMount:MountingHole_5mm_slot_no_keepout"
 			(at 330.2 129.54 0)
 			(effects
